File: Bluetooth_Board_STM32WB5MMGH6TR.kicad_pcb (KiCad board)
At the start: 4 copper layers, 50 x 50 mm, 69 parts, among them J1 Coin Battery Jumper, J10 3V3 Power Pins, J11 GPIO_Pin_Headers, J13 LPUART1_Header, J14 USART1_Header, J15 SPI1_Header, J16 SPI2_Header, J17 I2C1_Header, J18 QuadSPI_Headers, J19 I2C1_Header, J2 BOOT0_Jumper, J20 GPIO_Pin_Headers, J3 User Button Jumper, J4 USB_B_Micro, J5 Debug_Pins, J6 Power Select Jumpers, J7 3V3 Power Source Jumpers, J8 Power Pins, J9 5V Power Pins, U1 STM32WB5MMGH6TR, U5 USBLC6-2SC6

Commit message: Pins selected
Parts:
- removed J17, J19: I2C1_Header, Connector_PinHeader_2.54mm:PinHeader_1x04_P2.54mm_Vertical
- removed R19, R20, R21, R22, R23, R24: 100R, Resistor_SMD:R_0805_2012Metric_Pad1.20x1.40mm_HandSolder
- added J12: GPIO_Pin_Headers, Connector_PinHeader_2.54mm:PinHeader_2x13_P2.54mm_Vertical, F.Cu at (178.7, 27.1)
- BH1, C12, C3, C6, FB1: moved to B.Cu
- J11: value GPIO_Pin_Headers -> SPI1_Header; footprint Connector_PinHeader_2.54mm:PinHeader_2x11_P2.54mm_Vertical -> Connector_PinHeader_2.54mm:PinHeader_2x05_P2.54mm_Vertical
- J13: value LPUART1_Header -> I2C1_Header; footprint Connector_PinHeader_2.54mm:PinHeader_1x04_P2.54mm_Vertical -> Connector_PinHeader_2.54mm:PinHeader_2x03_P2.54mm_Vertical
- J14: value USART1_Header -> I2C1_Header; footprint Connector_PinHeader_2.54mm:PinHeader_1x04_P2.54mm_Vertical -> Connector_PinHeader_2.54mm:PinHeader_2x03_P2.54mm_Vertical
- J15: value SPI1_Header -> LPUART1_Header; footprint Connector_PinHeader_2.54mm:PinHeader_1x06_P2.54mm_Vertical -> Connector_PinHeader_2.54mm:PinHeader_2x03_P2.54mm_Vertical
- J16: value SPI2_Header -> USART1_Header; footprint Connector_PinHeader_2.54mm:PinHeader_1x06_P2.54mm_Vertical -> Connector_PinHeader_2.54mm:PinHeader_2x03_P2.54mm_Vertical
- J18: value QuadSPI_Headers -> GPIO_Pin_Headers; footprint Connector_PinHeader_2.54mm:PinHeader_1x08_P2.54mm_Vertical -> Connector_PinHeader_2.54mm:PinHeader_2x09_P2.54mm_Vertical
- J20: value GPIO_Pin_Headers -> SPI2_Header; footprint Connector_PinHeader_2.54mm:PinHeader_2x11_P2.54mm_Vertical -> Connector_PinHeader_2.54mm:PinHeader_2x05_P2.54mm_Vertical
- moved BH1 111.3 mm to (207.8, 46.9), turned to 90 degrees
- moved J20 94.8 mm to (62.1, 58.5)
- moved J18 68.5 mm to (83.1, 30.9)
- moved C10 54.3 mm to (150.3, 87.9)
- moved LDO1 54.3 mm to (147.2, 88.0)
- moved C9 54.3 mm to (144.1, 88.0)
- moved ESD2 43.6 mm to (146.2, 98.6)
- moved J11 35.5 mm to (54.9, 58.5)
- moved R13 31.8 mm to (96.3, 60.9)
- moved R14 31.8 mm to (96.3, 58.0)
- moved J2 25.5 mm to (100.0, 84.8)
- moved R1 24.9 mm to (97.1, 81.9)
- moved C5 23.2 mm to (105.1, 52.4), turned to 0 degrees
- moved U3 12.9 mm to (106.7, 59.4), turned to 90 degrees
- moved R4 8.80 mm to (168.8, 67.7)
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Connections:
- J11 pad 1: /PC12 -> +3.3V
- J11 pad 10: /PB14 -> GND
- J11 pad 2: /PB0 -> GND
- J11 pad 3: /PC13 -> Net-(J11-Pin_3)
- J11 pad 4: /PB1 -> GND
- J11 pad 5: /PA0 -> Net-(J11-Pin_5)
- J11 pad 6: /PB2 -> GND
- J11 pad 7: /PA3 -> Net-(J11-Pin_7)
- J11 pad 8: /PB12 -> GND
- J11 pad 9: unconnected-(J11-Pin_9-Pad9) -> Net-(J11-Pin_9)
- J13 pad 1: Net-(J13-Pin_1) -> +3.3V
- J13 pad 2: Net-(J13-Pin_2) -> GND
- J13 pad 3: GND -> Net-(J13-Pin_3)
- J13 pad 4: +3.3V -> GND
- J14 pad 4: Net-(J14-Pin_4) -> GND
- J15 pad 1: +3.3V -> Net-(J15-Pin_1)
- J15 pad 4: Net-(J15-Pin_4) -> GND
- J15 pad 5: Net-(J15-Pin_5) -> +3.3V
- J15 pad 6: Net-(J15-Pin_6) -> GND
- J16 pad 4: Net-(J16-Pin_4) -> GND
- J16 pad 6: Net-(J16-Pin_6) -> GND
- J18 pad 1: +3.3V -> /PA0
- J18 pad 2: GND -> /PB2
- J18 pad 3: Net-(J18-Pin_3) -> /PA3
- J18 pad 4: Net-(J18-Pin_4) -> /PB12
- J18 pad 5: Net-(J18-Pin_5) -> /PD4
- J18 pad 6: Net-(J18-Pin_6) -> /PB14
- J18 pad 7: Net-(J18-Pin_7) -> /PD5
- J18 pad 8: Net-(J18-Pin_8) -> /PB15
- J20 pad 1: /PD2 -> +3.3V
- J20 pad 10: /PC5 -> GND
- J20 pad 2: /PD13 -> GND
- J20 pad 3: /PD3 -> Net-(J20-Pin_3)
- J20 pad 4: /PD14 -> GND
- J20 pad 5: /PD6 -> Net-(J20-Pin_5)
- J20 pad 6: /PD15 -> GND
- J20 pad 7: /PD7 -> Net-(J20-Pin_7)
- J20 pad 8: /PC4 -> GND
- J20 pad 9: /PD8 -> Net-(J20-Pin_9)
- R10 pad 2: Net-(J16-Pin_4) -> Net-(J20-Pin_5)
- R11 pad 2: Net-(J16-Pin_5) -> Net-(J20-Pin_7)
- R12 pad 2: Net-(J16-Pin_6) -> Net-(J20-Pin_9)
- R13 pad 2: Net-(J19-Pin_3) -> Net-(J14-Pin_3)
- R14 pad 2: Net-(J19-Pin_4) -> Net-(J14-Pin_5)
- R15 pad 2: Net-(J17-Pin_3) -> Net-(J13-Pin_3)
- R16 pad 2: Net-(J17-Pin_4) -> Net-(J13-Pin_5)
- R17 pad 2: Net-(J14-Pin_3) -> Net-(J16-Pin_3)
- R18 pad 2: Net-(J14-Pin_4) -> Net-(J16-Pin_5)
- R2 pad 2: Net-(J13-Pin_1) -> Net-(J15-Pin_1)
- R3 pad 2: Net-(J13-Pin_2) -> Net-(J15-Pin_3)
- R4 pad 2: Net-(J15-Pin_3) -> Net-(J11-Pin_3)
- R6 pad 2: Net-(J15-Pin_4) -> Net-(J11-Pin_5)
- R7 pad 2: Net-(J15-Pin_5) -> Net-(J11-Pin_7)
- R8 pad 2: Net-(J15-Pin_6) -> Net-(J11-Pin_9)
- R9 pad 2: Net-(J16-Pin_3) -> Net-(J20-Pin_3)
- U1 pad 45: /PC5 -> unconnected-(U1-PC5-Pad45)
- U1 pad 46: /PB11_QUADSPI_BK1_NCS -> unconnected-(U1-PB11-Pad46)
- U1 pad 47: /PB10_QUADSPI_CLK -> unconnected-(U1-PB10-Pad47)
- U1 pad 52: /PA7_QUADSPI_BK1_IO2 -> /PA7
- U1 pad 53: /PA6_QUADSPI_BK1_IO3 -> /PA6
- U1 pad 72: GND -> /PE3
- U1 pad 73: /PD4_QUADSPI_BK1_IO0 -> /PD4
- U1 pad 80: /PD5_QUADSPI_BK1_IO1 -> /PD5
- U1 pad 83: GND -> /PC8
Routing:
- net /PC0_LPUART1_RX: track 0.00 -> 13.8 mm, vias 0 -> 1
- net /PB10_QUADSPI_CLK: track 13.4 -> 0.00 mm
- net /PH1: track 0.00 -> 13.4 mm, vias 0 -> 1
- net Net-(U1-PH3-BOOT0): track 0.00 -> 12.8 mm, vias 0 -> 1
- net /PB11_QUADSPI_BK1_NCS: track 12.7 -> 0.00 mm
- net /PD10: track 0.00 -> 12.3 mm, vias 0 -> 1
- net /PC5: track 12.1 -> 0.00 mm
- net /PB8_I2C1_SCL: track 0.00 -> 11.7 mm, vias 0 -> 1
- net /PC8: track 0.00 -> 11.3 mm, vias 0 -> 1
- net /PD4: track 0.00 -> 10.1 mm, vias 0 -> 1
- net /PB0: track 11.6 -> 1.54 mm, vias 0 -> 1
- net /PB1: track 10.9 -> 1.11 mm, vias 0 -> 1
- net /PE0: track 0.00 -> 9.44 mm, vias 0 -> 1
- net /PE3: track 0.00 -> 9.42 mm, vias 0 -> 1
- net /PD11: track 0.00 -> 9.33 mm, vias 0 -> 1
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- added copper zone on B.Cu, net GND
- added copper zone on In2.Cu, net GND
- added copper zone on In3.Cu, net GND
- added copper zone on In4.Cu, net GND
Other:
- copper layers 4 -> 6

Commit message: Update
Parts:
- removed C6: 100n, Capacitor_SMD:C_0805_2012Metric_Pad1.18x1.45mm_HandSolder
- removed ESD1, ESD2: ESDALC6V1W5, Personal_Project:SOT323-5L_STM-L
- removed J10: 3V3 Power Pins, Connector_PinHeader_2.54mm:PinHeader_2x03_P2.54mm_Vertical
- removed J15: LPUART1_Header, Connector_PinHeader_2.54mm:PinHeader_2x03_P2.54mm_Vertical
- removed J20: SPI2_Header, Connector_PinHeader_2.54mm:PinHeader_2x05_P2.54mm_Vertical
- removed J9: 5V Power Pins, Connector_PinHeader_2.54mm:PinHeader_2x03_P2.54mm_Vertical
- added J17: SAI1_B_Header, Connector_PinHeader_2.54mm:PinHeader_2x05_P2.54mm_Vertical, F.Cu at (156.0, 74.5)
- added J19: QUADSPI_Header, Connector_PinHeader_2.54mm:PinHeader_2x07_P2.54mm_Vertical, F.Cu at (84.5, 19.2)
- added R19: 100R, Resistor_SMD:R_0805_2012Metric_Pad1.20x1.40mm_HandSolder, F.Cu at (91.7, 18.4)
- added R20: 100R, Resistor_SMD:R_0805_2012Metric_Pad1.20x1.40mm_HandSolder, F.Cu at (91.7, 21.3)
- added R21: 100R, Resistor_SMD:R_0805_2012Metric_Pad1.20x1.40mm_HandSolder, F.Cu at (91.7, 24.3)
- added R22: 100R, Resistor_SMD:R_0805_2012Metric_Pad1.20x1.40mm_HandSolder, F.Cu at (91.7, 27.2)
- added R23: 100R, Resistor_SMD:R_0805_2012Metric_Pad1.20x1.40mm_HandSolder, F.Cu at (151.6, 76.7)
- added R24: 100R, Resistor_SMD:R_0805_2012Metric_Pad1.20x1.40mm_HandSolder, F.Cu at (151.6, 79.6)
- added R25: 100R, Resistor_SMD:R_0805_2012Metric_Pad1.20x1.40mm_HandSolder, F.Cu at (151.5, 82.2)
- added R26: 100R, Resistor_SMD:R_0805_2012Metric_Pad1.20x1.40mm_HandSolder, F.Cu at (151.5, 85.1)
- added R27: 100R, Resistor_SMD:R_0805_2012Metric_Pad1.20x1.40mm_HandSolder, F.Cu at (108.7, 17.7)
- added R28: 100R, Resistor_SMD:R_0805_2012Metric_Pad1.20x1.40mm_HandSolder, F.Cu at (108.7, 20.7)
- J12: value GPIO_Pin_Headers -> TIM1_CH1_Headers; footprint Connector_PinHeader_2.54mm:PinHeader_2x13_P2.54mm_Vertical -> Connector_PinHeader_2.54mm:PinHeader_2x02_P2.54mm_Vertical
- J13: value I2C1_Header -> SAI1_A_Header; footprint Connector_PinHeader_2.54mm:PinHeader_2x03_P2.54mm_Vertical -> Connector_PinHeader_2.54mm:PinHeader_2x05_P2.54mm_Vertical
- J18: value GPIO_Pin_Headers -> ADC1_Headers; footprint Connector_PinHeader_2.54mm:PinHeader_2x09_P2.54mm_Vertical -> Connector_PinHeader_2.54mm:PinHeader_2x02_P2.54mm_Vertical
- moved R10 108.5 mm to (79.6, 34.3)
- moved R9 108.5 mm to (79.6, 31.7)
- moved J11 100.8 mm to (155.7, 59.0)
- moved R2 98.9 mm to (173.6, 27.0)
- moved R3 98.9 mm to (173.6, 29.5)
- moved R14 56.7 mm to (130.8, 103.0), turned to -90 degrees
- moved R13 56.4 mm to (133.8, 103.0), turned to -90 degrees
- moved R16 53.9 mm to (161.4, 135.3), turned to 0 degrees
- moved R15 51.3 mm to (161.4, 132.3), turned to 0 degrees
- moved J18 32.7 mm to (113.0, 17.7)
- moved R18 26.6 mm to (154.6, 109.8), turned to 0 degrees
- moved R17 23.2 mm to (154.5, 107.0), turned to 0 degrees
- moved R4 18.3 mm to (151.8, 60.9)
- moved R6 18.3 mm to (151.8, 63.8)
- moved R8 18.3 mm to (151.8, 69.7)
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Connections:
- J12 pad 1: /PD2 -> Net-(J12-Pin_1)
- J12 pad 2: /PD13 -> GND
- J12 pad 3: /PD3 -> Net-(J12-Pin_3)
- J12 pad 4: /PD14 -> GND
- J18 pad 1: /PA0 -> Net-(J18-Pin_1)
- J18 pad 2: /PB2 -> GND
- J18 pad 3: /PA3 -> Net-(J18-Pin_3)
- J18 pad 4: /PB12 -> GND
- J3 pad 2: /PD2 -> /PA1_USR_BTN
- R10 pad 1: /PC3_SPI2_MOSI -> /PD7_QUADSPI_BK1_IO3
- R11 pad 1: /PD0_SPI2_NSS -> /PB12_SAI1_FS_A
- R11 pad 2: Net-(J20-Pin_7) -> Net-(J13-Pin_3)
- R12 pad 1: /PD1_SPI2_SCK -> /PB13_SAI1_SCK_A
- R12 pad 2: Net-(J20-Pin_9) -> Net-(J13-Pin_5)
- R14 pad 1: /PB9_I2C1_SDA -> /PA10_I2C1_SDA
- R15 pad 1: /PC1_I2C3_SDA -> /PB15_SAI1_SD_A
- R15 pad 2: Net-(J13-Pin_3) -> Net-(J13-Pin_7)
- R16 pad 1: /PB13_I2C3_SCL -> /PB14_SAI1_MCLK_A
- R16 pad 2: Net-(J13-Pin_5) -> Net-(J13-Pin_9)
- R18 pad 1: /PC0_LPUART1_RX -> /PB10_LPUART1_RX
- R2 pad 1: /PB6_USART1_TX -> /PA0_TIM2_CH1
- R2 pad 2: Net-(J15-Pin_1) -> Net-(J12-Pin_1)
- R3 pad 1: /PB7_USART1_RX -> /PD14_TIM1_CH1
- R3 pad 2: Net-(J15-Pin_3) -> Net-(J12-Pin_3)
- R4 pad 1: /PA1_SPI1_SCK -> /PA5_SPI1_SCK
- R7 pad 1: /PB4_SPI1_MISO -> /PA6_SPI1_MISO
- R8 pad 1: /PB5_SPI1_MOSI -> /PA7_SPI1_MOSI
- R9 pad 1: /PC2_SPI2_MISO -> /PD6_QUADSPI_BK1_IO2
- U1 pad 11: /PB9_I2C1_SDA -> /PB9_QUADSPI_BK1_IO0
- U1 pad 12: /PC0_LPUART1_RX -> /PC0_ADC1_IN1
- U1 pad 18: /PB7_USART1_RX -> unconnected-(U1-PB7-Pad18)
- U1 pad 19: /PB5_SPI1_MOSI -> /PB5_SAI1_SD_B
- U1 pad 2: /PA1_SPI1_SCK -> /PA1_USR_BTN
- U1 pad 20: /PB4_SPI1_MISO -> /PB4_SAI1_MCLK_B
- U1 pad 22: /PC10 -> unconnected-(U1-PC10-Pad22)
- U1 pad 23: /PC11 -> unconnected-(U1-PC11-Pad23)
- U1 pad 24: /PC12 -> unconnected-(U1-PC12-Pad24)
- U1 pad 28: /PA10 -> /PA10_I2C1_SDA
- U1 pad 3: /PA0 -> /PA0_TIM2_CH1
- U1 pad 33: /PD0_SPI2_NSS -> unconnected-(U1-PD0-Pad33)
- U1 pad 34: /PD1_SPI2_SCK -> unconnected-(U1-PD1-Pad34)
- U1 pad 35: /PB13_I2C3_SCL -> /PB13_SAI1_SCK_A
- U1 pad 36: /PC6 -> unconnected-(U1-PC6-Pad36)
- U1 pad 37: /PB14 -> /PB14_SAI1_MCLK_A
- U1 pad 38: /PB15 -> /PB15_SAI1_SD_A
- U1 pad 39: /PB6_USART1_TX -> unconnected-(U1-PB6-Pad39)
- U1 pad 4: +3.3V -> Net-(U1-VDDA)
- U1 pad 40: /PC13 -> unconnected-(U1-PC13-Pad40)
- U1 pad 41: /PB12 -> /PB12_SAI1_FS_A
- U1 pad 42: /PE4 -> unconnected-(U1-PE4-Pad42)
- U1 pad 43: /PB1 -> unconnected-(U1-PB1-Pad43)
- U1 pad 44: /PB0 -> unconnected-(U1-PB0-Pad44)
- U1 pad 46: unconnected-(U1-PB11-Pad46) -> /PB11_QUADSPI_BK1_NCS
- U1 pad 47: unconnected-(U1-PB10-Pad47) -> /PB10_LPUART1_RX
- U1 pad 48: /PB2 -> unconnected-(U1-PB2-Pad48)
- U1 pad 49: /PC4 -> unconnected-(U1-PC4-Pad49)
- U1 pad 50: /PA8 -> unconnected-(U1-PA8-Pad50)
- U1 pad 51: /PA9 -> unconnected-(U1-PA9-Pad51)
- U1 pad 52: /PA7 -> /PA7_SPI1_MOSI
- U1 pad 53: /PA6 -> /PA6_SPI1_MISO
- U1 pad 54: unconnected-(U1-PA5-Pad54) -> /PA5_SPI1_SCK
- U1 pad 55: unconnected-(U1-PA4-Pad55) -> /PA4_SAI1_FS_B
- U1 pad 56: /PA3 -> /PA3_QUADSPI_CLK
- U1 pad 61: /PH0 -> unconnected-(U1-PH0-Pad61)
- U1 pad 62: /PH1 -> unconnected-(U1-PH1-Pad62)
- U1 pad 63: /PD14 -> /PD14_TIM1_CH1
- U1 pad 64: /PE1 -> unconnected-(U1-PE1-Pad64)
- U1 pad 65: /PD13 -> unconnected-(U1-PD13-Pad65)
- U1 pad 66: /PD12 -> unconnected-(U1-PD12-Pad66)
- U1 pad 67: /PD7 -> /PD7_QUADSPI_BK1_IO3
- U1 pad 68: /PD2 -> unconnected-(U1-PD2-Pad68)
- U1 pad 69: /PC9 -> /PC9_SAI1_SCK_B
- U1 pad 7: /PC3_SPI2_MOSI -> unconnected-(U1-PC3-Pad7)
- U1 pad 70: /PD3 -> unconnected-(U1-PD3-Pad70)
- U1 pad 71: /PC7 -> unconnected-(U1-PC7-Pad71)
- U1 pad 72: /PE3 -> unconnected-(U1-PE3-Pad72)
- U1 pad 73: /PD4 -> unconnected-(U1-PD4-Pad73)
- U1 pad 74: /PD9 -> unconnected-(U1-PD9-Pad74)
- U1 pad 75: /PD8 -> unconnected-(U1-PD8-Pad75)
- U1 pad 76: /PD15 -> unconnected-(U1-PD15-Pad76)
- U1 pad 77: /PD10 -> unconnected-(U1-PD10-Pad77)
- U1 pad 78: /PE2 -> unconnected-(U1-PE2-Pad78)
- U1 pad 79: /PE0 -> unconnected-(U1-PE0-Pad79)
- U1 pad 8: /PC2_SPI2_MISO -> unconnected-(U1-PC2-Pad8)
- U1 pad 80: /PD5 -> /PD5_QUADSPI_BK1_IO1
- U1 pad 81: /PD6 -> /PD6_QUADSPI_BK1_IO2
- U1 pad 82: /PD11 -> unconnected-(U1-PD11-Pad82)
- U1 pad 83: /PC8 -> unconnected-(U1-PC8-Pad83)
- U1 pad 9: /PC1_I2C3_SDA -> /PC1_ADC1_IN2
Routing:
- net unconnected-(U1-PC2-Pad8): track 0.00 -> 15.7 mm, vias 0 -> 1
- net /PC2_SPI2_MISO: track 15.7 -> 0.00 mm, vias 1 -> 0
- net /PC1_I2C3_SDA: track 14.9 -> 0.00 mm, vias 1 -> 0
- net /PC1_ADC1_IN2: track 0.00 -> 14.9 mm, vias 0 -> 1
- net /PB9_QUADSPI_BK1_IO0: track 0.00 -> 14.5 mm, vias 0 -> 1
- net /PB9_I2C1_SDA: track 14.5 -> 0.00 mm, vias 1 -> 0
- net /PA0_TIM2_CH1: track 0.00 -> 14.1 mm, vias 0 -> 1
- net /PA0: track 14.1 -> 0.00 mm, vias 1 -> 0
- net /PC0_LPUART1_RX: track 13.8 -> 0.00 mm, vias 1 -> 0
- net /PC0_ADC1_IN1: track 0.00 -> 13.8 mm, vias 0 -> 1
- net unconnected-(U1-PH1-Pad62): track 0.00 -> 13.4 mm, vias 0 -> 1
- net /PH1: track 13.4 -> 0.00 mm, vias 1 -> 0
- net unconnected-(U1-PC3-Pad7): track 0.00 -> 12.5 mm, vias 0 -> 1
- net /PC3_SPI2_MOSI: track 12.5 -> 0.00 mm, vias 1 -> 0
- net unconnected-(U1-PD10-Pad77): track 0.00 -> 12.3 mm, vias 0 -> 1
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
Commit message: Update
Parts:
- removed C11, C8: 4u7, Capacitor_SMD:C_0603_1608Metric_Pad1.08x0.95mm_HandSolder
- removed J3: User Button Jumper, Connector_PinHeader_2.54mm:PinHeader_1x02_P2.54mm_Vertical
- removed J5: Debug_Pins, Connector_PinHeader_2.54mm:PinHeader_2x04_P2.54mm_Vertical
- removed J8: Power Pins, Connector_PinHeader_2.54mm:PinHeader_1x04_P2.54mm_Vertical
- removed R13, R14: 100R, Resistor_SMD:R_0805_2012Metric_Pad1.20x1.40mm_HandSolder
- added C13: 4u7, Capacitor_SMD:C_0603_1608Metric_Pad1.08x0.95mm_HandSolder, F.Cu at (151.1, 83.5)
- added C6: 4u7, Capacitor_SMD:C_0603_1608Metric_Pad1.08x0.95mm_HandSolder, F.Cu at (125.0, 83.8)
- added ESD1: ESDALC6V1W5, Personal_Project:SOT323-5L_STM-L, F.Cu at (151.0, 89.8)
- added J10: 5V_Selection_Header, Connector_PinHeader_2.54mm:PinHeader_1x03_P2.54mm_Vertical, F.Cu at (152.7, 86.2)
- added J9: 3V_Selection_Header, Connector_PinHeader_2.54mm:PinHeader_1x03_P2.54mm_Vertical, F.Cu at (126.7, 86.7)
- J16: value USART1_Header -> LPUART1_Header
- J6: value Power Select Jumpers -> Power_Pins; footprint Personal_Project:PinHeader_2x03_P2.54mm_Vertical_PINS -> Connector_PinHeader_2.54mm:PinHeader_1x03_P2.54mm_Vertical
- J7: value 3V3 Power Source Jumpers -> SWD_Pins; footprint Personal_Project:PinHeader_2x03_P2.54mm_Vertical_PINS -> Connector_PinHeader_2.54mm:PinHeader_1x05_P2.54mm_Horizontal
- moved U2 84.2 mm to (160.9, 88.2), turned to 90 degrees
- moved C2 74.2 mm to (159.4, 81.7)
- moved J6 67.7 mm to (152.8, 93.4), turned to -90 degrees
- moved J7 36.5 mm to (133.5, 92.0), turned to -90 degrees
- moved C5 31.1 mm to (116.8, 81.2)
- moved U3 31.0 mm to (118.3, 88.1)
- moved C10 19.5 mm to (130.8, 86.8), turned to 90 degrees
- moved J17 18.3 mm to (171.9, 65.5)
- moved R23 18.3 mm to (167.5, 67.6)
- moved R24 18.3 mm to (167.5, 70.6)
- moved R25 18.3 mm to (167.4, 73.1)
- moved R26 18.3 mm to (167.4, 76.1)
- moved LDO1 13.5 mm to (133.8, 86.8), turned to 180 degrees
- moved C9 7.31 mm to (136.9, 86.8), turned to 90 degrees
- moved R5 3.27 mm to (144.1, 90.1), turned to 180 degrees
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Connections:
- C2 pad 2: Net-(J3-Pin_1) -> /PA1_USR_BTN
- J14 pad 3: Net-(J14-Pin_3) -> /PB8_I2C1_SCL
- J14 pad 5: Net-(J14-Pin_5) -> /PA10_I2C1_SDA
- J4 pad 1: /VBUS -> /VBUS_5V
- J6 pad 1: /VBUS -> /EXT_5V
- J6 pad 2: /PC_5V -> /EXT_3V3
- J6 pad 3: /5V_SW -> GND
- J7 pad 1: /LD_OUT_3V3 -> /JTMS-SWDIO
- J7 pad 2: /PC_3V3 -> /JTCK-SWCLK
- J7 pad 3: /3V3_SW -> /JTDO-TRACE-SWO
- J7 pad 4: +3.3V -> /NRST
- J7 pad 5: +3.3V -> GND
- U2 pad 1: Net-(J3-Pin_1) -> /PA1_USR_BTN
- U2 pad 2: Net-(J3-Pin_1) -> /PA1_USR_BTN
- U5 pad 5: /VBUS -> /VBUS_5V
Routing:
- net /VBUS_5V: track 0.00 -> 19.1 mm, vias 0 -> 2
- net /EXT_5V: track 0.00 -> 8.76 mm
- net Net-(J4-ID): track 0.00 -> 3.15 mm
Other:
- board text added: "G/NR/SO/SC/SIO"
- board text added: "GN/3V3/5V"
- board text added: "NRST"
- board text added: "USR BTN"

Commit message: update
Parts:
- removed C13, C6: 4u7, Capacitor_SMD:C_0603_1608Metric_Pad1.08x0.95mm_HandSolder
- removed ESD1: ESDALC6V1W5, Personal_Project:SOT323-5L_STM-L
- removed J10: 5V_Selection_Header, Connector_PinHeader_2.54mm:PinHeader_1x03_P2.54mm_Vertical
- removed J6: Power_Pins, Connector_PinHeader_2.54mm:PinHeader_1x03_P2.54mm_Vertical
- removed J9: 3V_Selection_Header, Connector_PinHeader_2.54mm:PinHeader_1x03_P2.54mm_Vertical
- added C8: 4u7, Capacitor_SMD:C_0603_1608Metric_Pad1.08x0.95mm_HandSolder, F.Cu at (188.4, 101.3)
- added D1: BZX84C4V3LT1G, Package_TO_SOT_SMD:SOT-23, F.Cu at (188.7, 93.2)
- added D2: BZX84C6V2LT1G, Package_TO_SOT_SMD:SOT-23, F.Cu at (188.7, 97.8)
- added J3: JST_XH_2.54_Plug, Personal_Project:Connector_Power2pin_SHDRRA2W80P0X250_1X2_740X1150X610P, F.Cu at (175.7, 93.2)
- added J5: Power_Selector_Jumper, Connector_PinHeader_2.54mm:PinHeader_2x03_P2.54mm_Vertical, F.Cu at (174.7, 97.8)
- added J8: 3V_Selection_Header, Connector_PinHeader_2.54mm:PinHeader_1x03_P2.54mm_Vertical, F.Cu at (183.9, 93.1)
- added Q1: MOSFET_SI2333DDS-T1-BE3, Personal_Project:MOSFET_ SI2333DDS_SOT_DS-T1-BE3_VIS, F.Cu at (193.5, 93.3)
- added R13: 100k, Resistor_SMD:R_0603_1608Metric_Pad0.98x0.95mm_HandSolder, F.Cu at (188.4, 103.8)
- added S1: Switch_WS-SLSU SMT Mini Slide, Personal_Project:Switch_WS-SLSU SMT Mini Slide, F.Cu at (186.7, 86.7)
- added Z1: Diode_BZX84C6V2-7-F, Personal_Project:Diode_BZX84C6V2_SOT96P240X110-3N, F.Cu at (192.9, 102.3)
Routing:
- net /EXT_5V: track 8.76 -> 0.00 mm

Commit message: Update
Parts:
- removed BH1: Battery_Holder_1060TR, Personal_Project:Battery_Holder_1060TR
- removed C1: 100n, Capacitor_SMD:C_0805_2012Metric_Pad1.18x1.45mm_HandSolder
- removed J1: Coin Battery Jumper, Connector_PinHeader_2.54mm:PinHeader_1x03_P2.54mm_Vertical
- added J10: SPI1_Headers, Connector_PinHeader_2.54mm:PinHeader_2x03_P2.54mm_Horizontal, F.Cu at (215.8, 56.1)
- added J15: General_Pin_Header, Connector_PinHeader_2.54mm:PinHeader_2x03_P2.54mm_Horizontal, F.Cu at (215.8, 65.8)
- added J6: I2C1_Headers, Connector_PinHeader_2.54mm:PinHeader_2x03_P2.54mm_Horizontal, F.Cu at (215.8, 36.7)
- added J9: LPUART1_Headers, Connector_PinHeader_2.54mm:PinHeader_2x03_P2.54mm_Horizontal, F.Cu at (215.8, 46.4)
- added R14: 33R, Resistor_SMD:R_0805_2012Metric, F.Cu at (231.7, 35.8)
- added R29: 33R, Resistor_SMD:R_0805_2012Metric, F.Cu at (231.7, 38.8)
- added R30: 33R, Resistor_SMD:R_0805_2012Metric, F.Cu at (231.7, 41.7)
- added R31: 33R, Resistor_SMD:R_0805_2012Metric, F.Cu at (231.7, 44.7)
- added R32: 33R, Resistor_SMD:R_0805_2012Metric, F.Cu at (231.7, 47.6)
- moved J3 55.3 mm to (120.9, 85.2), turned to 90 degrees
- moved C5 9.66 mm to (117.2, 71.5)
- moved U3 9.66 mm to (118.7, 78.5)
- moved C9 8.90 mm to (145.8, 86.8)
- moved R5 8.90 mm to (153.0, 90.1)
- moved U5 8.90 mm to (149.3, 88.1)
- moved J4 8.90 mm to (149.7, 93.7)
Connections:
- U1 pad 15: /VBAT -> +3.3V
Routing:
- net unconnected-(U1-PB0-Pad44): track 1.54 -> 4.42 mm
- net /VBAT: track 1.02 -> 0.00 mm, vias 1 -> 0
- net +3.3V: track 2.83 -> 3.85 mm, vias 1 -> 2
