File: Bluetooth_Board_STM32WB5MMGH6TR.kicad_sch (KiCad schematic)
At the start: 67 parts, among them J1 Coin Battery Jumper, J10 3V3 Power Pins, J11 GPIO_Pin_Headers, J13 LPUART1_Header, J14 USART1_Header, J15 SPI1_Header, J16 SPI2_Header, J17 I2C1_Header, J18 QuadSPI_Headers, J19 I2C1_Header, J2 BOOT0_Jumper, J20 GPIO_Pin_Headers, J3 User Button Jumper, J4 USB_B_Micro, J5 Debug_Pins, J6 Power Select Jumpers, J7 3V3 Power Source Jumpers, J8 Power Pins, J9 5V Power Pins, U1 STM32WB5MMGH6TR, U5 USBLC6-2SC6

Commit message: Update
Parts:
- added C12: 4u7, Capacitor_SMD:C_0805_2012Metric_Pad1.18x1.45mm_HandSolder, symbol Device:C
- added FB1: BLM21PG601SN1D_0805, Capacitor_SMD:C_0805_2012Metric_Pad1.18x1.45mm_HandSolder, symbol Device:FerriteBead
- C3, C4, C6, C7: footprint (none) -> Capacitor_SMD:C_0805_2012Metric_Pad1.18x1.45mm_HandSolder
- J11, J20: footprint (none) -> Connector_PinHeader_2.54mm:PinHeader_2x11_P2.54mm_Vertical
- J13: footprint Connector_PinHeader_2.54mm:PinHeader_1x04_P2.54mm_Horizontal -> Connector_PinHeader_2.54mm:PinHeader_1x04_P2.54mm_Vertical
- J15, J16: footprint Connector_PinHeader_2.54mm:PinHeader_1x06_P2.54mm_Horizontal -> Connector_PinHeader_2.54mm:PinHeader_1x06_P2.54mm_Vertical
- J18: footprint (none) -> Connector_PinHeader_2.54mm:PinHeader_1x08_P2.54mm_Vertical
Connections:
- net PA1 is gone; now on net PD2: J3.2 (Pin_2)
- net PA13_SWDIO is gone; now on net JTMS-SWDIO: J5.2 (Pin_2)
- net PA14_SWCLK is gone; now on net JTCK-SWCLK: J5.4 (Pin_4)
- net PB3_SWO is gone; now on net JTDO-TRACE-SWO: J5.6 (Pin_6)
- net +3.3V: now also FB1.1; no longer C7.1, U1.6 (VDDA)
- net GND: now also U1.72 (PE3), U1.83 (PC8), C12.2
- net PA4: no longer names the net of U1.55 (PA4)
- net PA4: no longer J11.9 (Pin_9)
- net PA5: no longer names the net of U1.54 (PA5)
- net PA5: no longer J11.11 (Pin_11)
- net PC8: no longer names the net of J20.16 (Pin_16)
- net PC8: no longer U1.83 (PC8)
- net PE3: no longer names the net of J11.19 (Pin_19)
- net PE3: no longer U1.72 (PE3)
- new net: C12.1, C7.1, FB1.2, U1.6 (VDDA)
- no-connect marks 3 -> 9
Other:
- note added: "The module contains STM32WB55VGY It includes clocks and a chip antenna Decoupling capacitors are part of the module PE3 and PC8 connectedd to GND to allow for a grounding pin to reach ground. Set them up as INPUTS. PA0 as a WKUP pin"
- note removed: "The module contains STM32WB55VGY It includes clocks and a chip antenna Decoupling capacitors are part of the module"

Commit message: Pins selected
Parts:
- removed C6: 100n, Capacitor_SMD:C_0805_2012Metric_Pad1.18x1.45mm_HandSolder, symbol Device:C
- removed ESD1, ESD2: ESDALC6V1W5, Personal_Project:SOT323-5L_STM-L, symbol Personal_Projects:ESDALC6V1W5
- removed J11, J20: GPIO_Pin_Headers, Connector_PinHeader_2.54mm:PinHeader_2x11_P2.54mm_Vertical, symbol Connector_Generic:Conn_02x11_Odd_Even
- removed J13: LPUART1_Header, Connector_PinHeader_2.54mm:PinHeader_1x04_P2.54mm_Vertical, symbol Connector_Generic:Conn_01x04
- removed J14: USART1_Header, Connector_PinHeader_2.54mm:PinHeader_1x04_P2.54mm_Vertical, symbol Connector_Generic:Conn_01x04
- removed J15: SPI1_Header, Connector_PinHeader_2.54mm:PinHeader_1x06_P2.54mm_Vertical, symbol Connector_Generic:Conn_01x06
- removed J16: SPI2_Header, Connector_PinHeader_2.54mm:PinHeader_1x06_P2.54mm_Vertical, symbol Connector_Generic:Conn_01x06
- removed J17, J19: I2C1_Header, Connector_PinHeader_2.54mm:PinHeader_1x04_P2.54mm_Vertical, symbol Connector_Generic:Conn_01x04
- removed J18: QuadSPI_Headers, Connector_PinHeader_2.54mm:PinHeader_1x08_P2.54mm_Vertical, symbol Connector_Generic:Conn_01x08
- removed R2, R3: 100R, Resistor_SMD:R_0805_2012Metric_Pad1.20x1.40mm_HandSolder, symbol Device:R
- added J11: SPI1_Header, Connector_PinHeader_2.54mm:PinHeader_2x05_P2.54mm_Vertical, symbol Connector_Generic:Conn_02x05_Odd_Even
- added J13: SAI1_A_Header, Connector_PinHeader_2.54mm:PinHeader_2x05_P2.54mm_Vertical, symbol Connector_Generic:Conn_02x05_Odd_Even
- added J14: I2C1_Header, Connector_PinHeader_2.54mm:PinHeader_2x03_P2.54mm_Vertical, symbol Connector_Generic:Conn_02x03_Odd_Even
- added J16: USART1_Header, Connector_PinHeader_2.54mm:PinHeader_2x03_P2.54mm_Vertical, symbol Connector_Generic:Conn_02x03_Odd_Even
- added J17: SAI1_B_Header, Connector_PinHeader_2.54mm:PinHeader_2x05_P2.54mm_Vertical, symbol Connector_Generic:Conn_02x05_Odd_Even
- added J19: QUADSPI_Header, symbol Connector_Generic:Conn_02x07_Odd_Even
- added R25, R26: 100R, Resistor_SMD:R_0805_2012Metric_Pad1.20x1.40mm_HandSolder, symbol Device:R
Connections:
- net +3.3V: now also J11.1 (Pin_1), J13.1 (Pin_1), J14.1 (Pin_1), J16.1 (Pin_1), J17.1 (Pin_1), J19.1 (Pin_1); no longer U1.4 (VREF)
- net GND: now also J11.10 (Pin_10), J11.2 (Pin_2), J11.4 (Pin_4), J11.6 (Pin_6), J11.8 (Pin_8), J13.10 (Pin_10), J13.2 (Pin_2), J13.4 (Pin_4), J13.6 (Pin_6), J13.8 (Pin_8), J14.2 (Pin_2), J14.4 (Pin_4), J14.6 (Pin_6), J16.2 (Pin_2), J16.4 (Pin_4), J16.6 (Pin_6), J17.10 (Pin_10), J17.2 (Pin_2), J17.4 (Pin_4), J17.6 (Pin_6), J17.8 (Pin_8), J19.10 (Pin_10), J19.12 (Pin_12), J19.14 (Pin_14), J19.2 (Pin_2), J19.4 (Pin_4), J19.6 (Pin_6), J19.8 (Pin_8); no longer U1.72 (PE3), U1.83 (PC8)
- net PB11_QUADSPI_BK1_NCS: now also R20.1; no longer R24.1
- net at R21.2: now also J19.7 (Pin_7)
- net at R18.2: now also J16.5 (Pin_5)
- net at R17.2: now also J16.3 (Pin_3)
- net at R15.2: now also J13.7 (Pin_7)
- net at R16.2: now also J13.9 (Pin_9)
- net at C12.1, C7.1, FB1.2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: now also U1.4 (VREF)
- net at R8.2: now also J11.9 (Pin_9)
- net at R7.2: now also J11.7 (Pin_7)
- net at R20.2: now also J19.5 (Pin_5)
- net at R22.2: now also J19.9 (Pin_9)
- net at R4.2: now also J11.3 (Pin_3)
- net at R6.2: now also J11.5 (Pin_5)
- net at R24.2: now also J17.5 (Pin_5)
- net at R13.2: now also J14.3 (Pin_3)
- net at R12.2: now also J13.5 (Pin_5)
- net at R23.2: now also J17.3 (Pin_3)
- net at R14.2: now also J14.5 (Pin_5)
- net PA5_SPI1_SCK: now reaches U1.54 (PA5)
- net PA5_SPI1_SCK: now also R4.1
- net PA4_SAI1_FS_B: now reaches U1.55 (PA4)
- net PA4_SAI1_FS_B: now also R23.1
- net at R19.2: now also J19.3 (Pin_3)
- net at R11.2: now also J13.3 (Pin_3)
- net at R9.2: now also J19.11 (Pin_11)
- net at R10.2: now also J19.13 (Pin_13)
- net PA0 renamed PA0_TIM2_CH1
- net PA10 renamed PA10_I2C1_SDA
- net PA10_I2C1_SDA: now also R14.1
- net PA1_SPI1_SCK renamed PA1_USR_BTN
- net PA1_USR_BTN: now also J3.2 (Pin_2); no longer R4.1
- net PA3 renamed PA3_QUADSPI_CLK
- net PA3_QUADSPI_CLK: now also R19.1
- net PA6_QUADSPI_BK1_IO3 renamed PA6_SPI1_MISO
- net PA6_SPI1_MISO: now also R7.1; no longer R19.1
- net PA7_QUADSPI_BK1_IO2 renamed PA7_SPI1_MOSI
- net PA7_SPI1_MOSI: now also R8.1; no longer R20.1
- net PA8 renamed PA8_TIM1_CH1
- net PA9: no longer names the net of U1.51 (PA9)
- net PB0: no longer names the net of U1.44 (PB0)
- net PB1: no longer names the net of U1.43 (PB1)
- net PB10_QUADSPI_CLK renamed PB10_LPUART1_RX
- net PB10_LPUART1_RX: now also R18.1; no longer R23.1
- net PB12 renamed PB12_SAI1_FS_A
- net PB12_SAI1_FS_A: now also R11.1
- net PB13_I2C3_SCL renamed PB13_SAI1_SCK_A
- net PB13_SAI1_SCK_A: now also R12.1; no longer R16.1
- net PB14 renamed PB14_SAI1_MCLK_A
- net PB14_SAI1_MCLK_A: now also R16.1
- net PB15 renamed PB15_SAI1_SD_A
- net PB15_SAI1_SD_A: now also R15.1
- net PB2: no longer names the net of U1.48 (PB2)
- net PB4_SPI1_MISO renamed PB4_SAI1_MCLK_B
- net PB4_SAI1_MCLK_B: now also R26.1; no longer R7.1
- net PB5_SPI1_MOSI renamed PB5_SAI1_SD_B
- net PB5_SAI1_SD_B: now also R25.1; no longer R8.1
- net PB6_USART1_TX: no longer names the net of U1.39 (PB6)
- net PB7_USART1_RX: no longer names the net of U1.18 (PB7)
- net PB9_I2C1_SDA renamed PB9_QUADSPI_BK1_IO0
- net PB9_QUADSPI_BK1_IO0: now also R21.1; no longer R14.1
- net PC0_LPUART1_RX renamed PC0_ADC1_IN1
- net PC0_ADC1_IN1: no longer R18.1
- net PC10: no longer names the net of U1.22 (PC10)
- net PC11: no longer names the net of U1.23 (PC11)
- net PC12: no longer names the net of U1.24 (PC12)
- net PC13: no longer names the net of U1.40 (PC13)
- net PC1_I2C3_SDA renamed PC1_ADC1_IN2
- net PC1_ADC1_IN2: no longer R15.1
- net PC2_SPI2_MISO: no longer names the net of U1.8 (PC2)
- net PC2_SPI2_MISO: no longer R9.1
- net PC3_SPI2_MOSI: no longer names the net of U1.7 (PC3)
- net PC3_SPI2_MOSI: no longer R10.1
- net PC4: no longer names the net of U1.49 (PC4)
- net PC5: no longer names the net of U1.45 (PC5)
- net PC6: no longer names the net of U1.36 (PC6)
- net PC7: no longer names the net of U1.71 (PC7)
- net PC9 renamed PC9_SAI1_SCK_B
- net PC9_SAI1_SCK_B: now also R24.1
- net PD0_SPI2_NSS: no longer names the net of U1.33 (PD0)
- net PD0_SPI2_NSS: no longer R11.1
- net PD10: no longer names the net of U1.77 (PD10)
- net PD11: no longer names the net of U1.82 (PD11)
- net PD12: no longer names the net of U1.66 (PD12)
- net PD13: no longer names the net of U1.65 (PD13)
- net PD14 renamed PD14_TIM1_CH1
- net PD15: no longer names the net of U1.76 (PD15)
- net PD1_SPI2_SCK: no longer names the net of U1.34 (PD1)
- net PD1_SPI2_SCK: no longer R12.1
- net PD2: no longer names the net of U1.68 (PD2)
- net PD2: no longer J3.2 (Pin_2)
- net PD3: no longer names the net of U1.70 (PD3)
- net PD4_QUADSPI_BK1_IO0: no longer names the net of U1.73 (PD4)
- net PD4_QUADSPI_BK1_IO0: no longer R21.1
- net PD6 renamed PD6_QUADSPI_BK1_IO2
- net PD6_QUADSPI_BK1_IO2: now also R9.1
- net PD7 renamed PD7_QUADSPI_BK1_IO3
- net PD7_QUADSPI_BK1_IO3: now also R10.1
- net PD8: no longer names the net of U1.75 (PD8)
- net PD9: no longer names the net of U1.74 (PD9)
- net PE0: no longer names the net of U1.79 (PE0)
- net PE1: no longer names the net of U1.64 (PE1)
- net PE2: no longer names the net of U1.78 (PE2)
- net PE4: no longer names the net of U1.42 (PE4)
- net PH0: no longer names the net of U1.61 (PH0)
- net PH1: no longer names the net of U1.62 (PH1)
- new net: J17.7 (Pin_7), R25.2
- new net: J17.9 (Pin_9), R26.2
- no-connect marks 9 -> 37
Other:
- moved on the sheet: C11, C8, J6, J7, R13, R14

Commit message: Update
Parts:
- removed J10: 3V3 Power Pins, Connector_PinHeader_2.54mm:PinHeader_2x03_P2.54mm_Vertical, symbol Connector_Generic:Conn_02x03_Odd_Even
- removed J9: 5V Power Pins, Connector_PinHeader_2.54mm:PinHeader_2x03_P2.54mm_Vertical, symbol Connector_Generic:Conn_02x03_Odd_Even
- added J12: TIM1_CH1_Headers, Connector_PinHeader_2.54mm:PinHeader_2x02_P2.54mm_Vertical, symbol Connector_Generic:Conn_02x02_Odd_Even
- added J18: ADC1_Headers, Connector_PinHeader_2.54mm:PinHeader_2x02_P2.54mm_Vertical, symbol Connector_Generic:Conn_02x02_Odd_Even
- added R2, R27, R28, R3: 100R, Resistor_SMD:R_0805_2012Metric_Pad1.20x1.40mm_HandSolder, symbol Device:R
- J16: value USART1_Header -> LPUART1_Header
- J19: footprint (none) -> Connector_PinHeader_2.54mm:PinHeader_2x07_P2.54mm_Vertical
Connections:
- net GND: now also J12.2 (Pin_2), J12.4 (Pin_4), J18.2 (Pin_2), J18.4 (Pin_4)
- net PA0_TIM2_CH1: now also R2.1
- net PC0_ADC1_IN1: now also R27.1
- net PC1_ADC1_IN2: now also R28.1
- net PD14_TIM1_CH1: now also R3.1
- net PA8_TIM1_CH1: no longer names the net of U1.50 (PA8)
- new net: J12.3 (Pin_3), R3.2
- new net: J12.1 (Pin_1), R2.2
- new net: J18.3 (Pin_3), R28.2
- new net: J18.1 (Pin_1), R27.2
- no-connect marks 37 -> 38
Other:
- note removed: "The module contains STM32WB55VGY It includes clocks and a chip antenna Decoupling capacitors are part of the module PE3 and PC8 connectedd to GND to allow for a grounding pin to reach ground. Set them up as INPUTS. PA0 as a WKUP pin"
- moved on the sheet: J11, J13, J14, J16, J17, J19, R10, R11, R12, R13, R14, R15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

Commit message: Update
Parts:
- removed C11, C8: 4u7, Capacitor_SMD:C_0603_1608Metric_Pad1.08x0.95mm_HandSolder, symbol Device:C
- removed J3: User Button Jumper, Connector_PinHeader_2.54mm:PinHeader_1x02_P2.54mm_Vertical, symbol Connector_Generic:Conn_01x02
- removed J5: Debug_Pins, Connector_PinHeader_2.54mm:PinHeader_2x04_P2.54mm_Vertical, symbol Connector_Generic:Conn_02x04_Odd_Even
- removed J6: Power Select Jumpers, Personal_Project:PinHeader_2x03_P2.54mm_Vertical_PINS, symbol Connector_Generic:Conn_02x03_Top_Bottom
- removed J7: 3V3 Power Source Jumpers, Personal_Project:PinHeader_2x03_P2.54mm_Vertical_PINS, symbol Connector_Generic:Conn_02x03_Top_Bottom
- removed J8: Power Pins, Connector_PinHeader_2.54mm:PinHeader_1x04_P2.54mm_Vertical, symbol Connector:Conn_01x04_Pin
- removed R13, R14: 100R, Resistor_SMD:R_0805_2012Metric_Pad1.20x1.40mm_HandSolder, symbol Device:R
- added C13, C6: 4u7, Capacitor_SMD:C_0603_1608Metric_Pad1.08x0.95mm_HandSolder, symbol Device:C
- added ESD1: ESDALC6V1W5, Personal_Project:SOT323-5L_STM-L, symbol Personal_Projects:ESDALC6V1W5
- added J10: 5V_Selection_Header, Connector_PinHeader_2.54mm:PinHeader_1x03_P2.54mm_Vertical, symbol Connector_Generic:Conn_01x03
- added J6: Power_Pins, Connector_PinHeader_2.54mm:PinHeader_1x03_P2.54mm_Vertical, symbol Connector_Generic:Conn_01x03
- added J7: SWD_Pins, Connector_PinHeader_2.54mm:PinHeader_1x05_P2.54mm_Horizontal, symbol Connector_Generic:Conn_01x05
- added J9: 3V_Selection_Header, Connector_PinHeader_2.54mm:PinHeader_1x03_P2.54mm_Vertical, symbol Connector_Generic:Conn_01x03
Connections:
- net +3.3V: now also C6.1, J9.2 (Pin_2)
- net +5V: now also C13.1, J10.2 (Pin_2)
- net GND: now also C13.2, C6.2, ESD1.2 (GND), J6.3 (Pin_3), J7.5 (Pin_5)
- net JTCK-SWCLK: now also J7.2 (Pin_2)
- net JTDO-TRACE-SWO: now also J7.3 (Pin_3)
- net JTMS-SWDIO: now also J7.1 (Pin_1)
- net LD_OUT_3V3: now also J9.1 (Pin_1)
- net NRST: now also J7.4 (Pin_4)
- net PA10_I2C1_SDA: now also J14.5 (Pin_5)
- net PA1_USR_BTN: now also C2.2, U2.1, U2.2
- net PB8_I2C1_SCL: now also J14.3 (Pin_3)
- net VBUS renamed VBUS_5V
- net VBUS_5V: now also ESD1.5 (I/O4), J10.3 (Pin_3)
- new net EXT_3V3: ESD1.4 (I/O3), J6.2 (Pin_2), J9.3 (Pin_3)
- new net EXT_5V: ESD1.3 (I/O2), J10.1 (Pin_1), J6.1 (Pin_1)
- no-connect marks 38 -> 39

Commit message: update
Parts:
- removed C13, C6: 4u7, Capacitor_SMD:C_0603_1608Metric_Pad1.08x0.95mm_HandSolder, symbol Device:C
- removed ESD1: ESDALC6V1W5, Personal_Project:SOT323-5L_STM-L, symbol Personal_Projects:ESDALC6V1W5
- removed J10: 5V_Selection_Header, Connector_PinHeader_2.54mm:PinHeader_1x03_P2.54mm_Vertical, symbol Connector_Generic:Conn_01x03
- removed J6: Power_Pins, Connector_PinHeader_2.54mm:PinHeader_1x03_P2.54mm_Vertical, symbol Connector_Generic:Conn_01x03
- removed J9: 3V_Selection_Header, Connector_PinHeader_2.54mm:PinHeader_1x03_P2.54mm_Vertical, symbol Connector_Generic:Conn_01x03
- added C8: 4u7, Capacitor_SMD:C_0603_1608Metric_Pad1.08x0.95mm_HandSolder, symbol Device:C
- added D1: BZX84C4V3LT1G, Package_TO_SOT_SMD:SOT-23, symbol Diode:BZX84Cxx
- added D2: BZX84C6V2LT1G, Package_TO_SOT_SMD:SOT-23, symbol Diode:BZX84Cxx
- added J10: SPI1_Headers, Connector_PinHeader_2.54mm:PinHeader_2x03_P2.54mm_Horizontal, symbol Connector_Generic:Conn_02x03_Odd_Even
- added J15: General_Pin_Header, Connector_PinHeader_2.54mm:PinHeader_2x03_P2.54mm_Horizontal, symbol Connector_Generic:Conn_02x03_Odd_Even
- added J3: JST_XH_2.54_Plug, Personal_Project:Connector_Power2pin_SHDRRA2W80P0X250_1X2_740X1150X610P, symbol Personal_Projects:Connector_Power2pin_JST_XH_2.54_Plug
- added J5: Power_Selector_Jumper, Connector_PinHeader_2.54mm:PinHeader_2x03_P2.54mm_Vertical, symbol Connector_Generic:Conn_02x03_Odd_Even
- added J6: I2C1_Headers, Connector_PinHeader_2.54mm:PinHeader_2x03_P2.54mm_Horizontal, symbol Connector_Generic:Conn_02x03_Odd_Even
- added J8: 3V_Selection_Header, Connector_PinHeader_2.54mm:PinHeader_1x03_P2.54mm_Vertical, symbol Connector_Generic:Conn_01x03
- added J9: LPUART1_Headers, Connector_PinHeader_2.54mm:PinHeader_2x03_P2.54mm_Horizontal, symbol Connector_Generic:Conn_02x03_Odd_Even
- added Q1: MOSFET_SI2333DDS-T1-BE3, Personal_Project:MOSFET_ SI2333DDS_SOT_DS-T1-BE3_VIS, symbol Personal_Projects:MOSFET_SI2333DDS-T1-BE3
- added R13: 100k, Resistor_SMD:R_0603_1608Metric_Pad0.98x0.95mm_HandSolder, symbol Device:R
- added R14, R29, R30, R31, R32: 33R, Resistor_SMD:R_0805_2012Metric, symbol Device:R
- added S1: Switch_WS-SLSU SMT Mini Slide, Personal_Project:Switch_WS-SLSU SMT Mini Slide, symbol Personal_Projects:Switch_WS-SLSU SMT Mini Slide
- added Z1: Diode_BZX84C6V2-7-F, Personal_Project:Diode_BZX84C6V2_SOT96P240X110-3N, symbol Personal_Projects:Diode_BZX84C6V2-7-F
Connections:
- net +3.3V: now also S1.2
- net GND: now also C8.2, D1.1 (A), D2.1 (A), J10.2 (Pin_2), J10.6 (Pin_6), J15.1 (Pin_1), J15.4 (Pin_4), J15.5 (Pin_5), J3.1 (POWER-), J6.2 (Pin_2), J6.3 (Pin_3), J6.4 (Pin_4), J6.6 (Pin_6), J9.2 (Pin_2), J9.3 (Pin_3), J9.4 (Pin_4), J9.6 (Pin_6), R13.2
- net LD_OUT_3V3: now also J8.3 (Pin_3)
- net PA2_LPUART1_TX: now also R14.2
- net PB8_I2C1_SCL: now also J6.5 (Pin_5)
- net VBUS_5V: now also D2.3 (K), J5.5 (Pin_5)
- new net: J10.1 (Pin_1), R30.2
- new net: J10.5 (Pin_5), R31.2
- new net: J9.1 (Pin_1), R14.1
- new net: J9.5 (Pin_5), R29.2
- new net: J10.4 (Pin_4), R32.1
- new net EXT_POWER+: J3.2 (POWER+), Q1.3 (D)
- new net EXT_POWER+_NOLDO: J5.2 (Pin_2), J8.1 (Pin_1)
- new net EXT_POWER+_PP: D1.3 (K), J5.1 (Pin_1), J5.3 (Pin_3), Q1.2 (S), Z1.3 (K)
- new net LDO_IN: J5.4 (Pin_4), J5.6 (Pin_6)
- new net MOSFET_GATE: Q1.1 (G), R13.1, Z1.1 (A)
- new net PA0: J15.6 (Pin_6)
- new net PA1_SPI1_SCK: R31.1
- new net PA3_LPUART1_RX: R29.1
- new net PA4_SPI1_NSS: J15.3 (Pin_3)
- new net PA8_MCO: J15.2 (Pin_2)
- new net PB4_SPI1_MISO: R30.1
- new net PB5_SPI1_MOSI: R32.2
- new net PB7_I2C1_SDA: J6.1 (Pin_1)
- new net POWER_3V3: C8.1, J8.2 (Pin_2), S1.1
- no-connect marks 39 -> 43
Other:
- note added: "Chip Select pin on general pin header"
- note added: "Input voltage range: 1.45V to 5.5V"
- note added: "ON/OFF Switch"
- note added: "Overvoltage protection for the PMOSFET VGS (VGS max is 8V)"
- note added: "Polarity Protection"

Commit message: Update
Parts:
- removed BH1: Battery_Holder_1060TR, Personal_Project:Battery_Holder_1060TR, symbol Personal_Projects:Battery_Holder_1060TR
- removed C1, C3, C4, C7: 100n, Capacitor_SMD:C_0805_2012Metric_Pad1.18x1.45mm_HandSolder, symbol Device:C
- removed C10, C9: 1u, Capacitor_SMD:C_0603_1608Metric_Pad1.08x0.95mm_HandSolder, symbol Device:C
- removed C12: 4u7, Capacitor_SMD:C_0805_2012Metric_Pad1.18x1.45mm_HandSolder, symbol Device:C
- removed C5: 100nF, Capacitor_SMD:C_0805_2012Metric_Pad1.18x1.45mm_HandSolder, symbol Device:C
- removed C8: 4u7, Capacitor_SMD:C_0603_1608Metric_Pad1.08x0.95mm_HandSolder, symbol Device:C
- removed D1: BZX84C4V3LT1G, Package_TO_SOT_SMD:SOT-23, symbol Diode:BZX84Cxx
- removed D2: BZX84C6V2LT1G, Package_TO_SOT_SMD:SOT-23, symbol Diode:BZX84Cxx
- removed FB1: BLM21PG601SN1D_0805, Capacitor_SMD:C_0805_2012Metric_Pad1.18x1.45mm_HandSolder, symbol Device:FerriteBead
- removed H1, H2, H3, H4, H5: MountingHole_Pad, MountingHole:MountingHole_3.2mm_M3_Pad, symbol Mechanical:MountingHole_Pad
- removed J1: Coin Battery Jumper, Connector_PinHeader_2.54mm:PinHeader_1x03_P2.54mm_Vertical, symbol Connector_Generic:Conn_01x03
- removed J10: SPI1_Headers, Connector_PinHeader_2.54mm:PinHeader_2x03_P2.54mm_Horizontal, symbol Connector_Generic:Conn_02x03_Odd_Even
- removed J11: SPI1_Header, Connector_PinHeader_2.54mm:PinHeader_2x05_P2.54mm_Vertical, symbol Connector_Generic:Conn_02x05_Odd_Even
- removed J12: TIM1_CH1_Headers, Connector_PinHeader_2.54mm:PinHeader_2x02_P2.54mm_Vertical, symbol Connector_Generic:Conn_02x02_Odd_Even
- removed J13: SAI1_A_Header, Connector_PinHeader_2.54mm:PinHeader_2x05_P2.54mm_Vertical, symbol Connector_Generic:Conn_02x05_Odd_Even
- removed J14: I2C1_Header, Connector_PinHeader_2.54mm:PinHeader_2x03_P2.54mm_Vertical, symbol Connector_Generic:Conn_02x03_Odd_Even
- removed J15: General_Pin_Header, Connector_PinHeader_2.54mm:PinHeader_2x03_P2.54mm_Horizontal, symbol Connector_Generic:Conn_02x03_Odd_Even
- removed J16: LPUART1_Header, Connector_PinHeader_2.54mm:PinHeader_2x03_P2.54mm_Vertical, symbol Connector_Generic:Conn_02x03_Odd_Even
- removed J17: SAI1_B_Header, Connector_PinHeader_2.54mm:PinHeader_2x05_P2.54mm_Vertical, symbol Connector_Generic:Conn_02x05_Odd_Even
- removed J18: ADC1_Headers, Connector_PinHeader_2.54mm:PinHeader_2x02_P2.54mm_Vertical, symbol Connector_Generic:Conn_02x02_Odd_Even
- removed J19: QUADSPI_Header, Connector_PinHeader_2.54mm:PinHeader_2x07_P2.54mm_Vertical, symbol Connector_Generic:Conn_02x07_Odd_Even
- removed J2: BOOT0_Jumper, Connector_PinHeader_2.54mm:PinHeader_1x03_P2.54mm_Vertical, symbol Connector:Conn_01x03_Pin
- removed J3: JST_XH_2.54_Plug, Personal_Project:Connector_Power2pin_SHDRRA2W80P0X250_1X2_740X1150X610P, symbol Personal_Projects:Connector_Power2pin_JST_XH_2.54_Plug
- removed J4: USB_B_Micro, Connector_USB:USB_Micro-B_Molex-105017-0001, symbol Connector:USB_B_Micro
- removed J5: Power_Selector_Jumper, Connector_PinHeader_2.54mm:PinHeader_2x03_P2.54mm_Vertical, symbol Connector_Generic:Conn_02x03_Odd_Even
- removed J6: I2C1_Headers, Connector_PinHeader_2.54mm:PinHeader_2x03_P2.54mm_Horizontal, symbol Connector_Generic:Conn_02x03_Odd_Even
- removed J7: SWD_Pins, Connector_PinHeader_2.54mm:PinHeader_1x05_P2.54mm_Horizontal, symbol Connector_Generic:Conn_01x05
- removed J8: 3V_Selection_Header, Connector_PinHeader_2.54mm:PinHeader_1x03_P2.54mm_Vertical, symbol Connector_Generic:Conn_01x03
- removed J9: LPUART1_Headers, Connector_PinHeader_2.54mm:PinHeader_2x03_P2.54mm_Horizontal, symbol Connector_Generic:Conn_02x03_Odd_Even
- removed LDO1: LDO_TLV75733PDBVR, Personal_Project:LDO_SOT95P280X145-5N, symbol Personal_Projects:LDO_TLV75733PDBVR
- removed Q1: MOSFET_SI2333DDS-T1-BE3, Personal_Project:MOSFET_ SI2333DDS_SOT_DS-T1-BE3_VIS, symbol Personal_Projects:MOSFET_SI2333DDS-T1-BE3
- removed R1: 1k, Resistor_SMD:R_0805_2012Metric_Pad1.20x1.40mm_HandSolder, symbol Device:R
- removed R10, R11, R12, R15, R16, R17, R18, R19, R2, R20, R21, R22, R23, R24, R25, R26, R27, R28, R3, R4, R6, R7, R8, R9: 100R, Resistor_SMD:R_0805_2012Metric_Pad1.20x1.40mm_HandSolder, symbol Device:R
- removed R13, R5: 100k, Resistor_SMD:R_0603_1608Metric_Pad0.98x0.95mm_HandSolder, symbol Device:R
- removed R14, R29, R30, R31, R32: 33R, Resistor_SMD:R_0805_2012Metric, symbol Device:R
- removed S1: Switch_WS-SLSU SMT Mini Slide, Personal_Project:Switch_WS-SLSU SMT Mini Slide, symbol Personal_Projects:Switch_WS-SLSU SMT Mini Slide
- removed U1: STM32WB5MMGH6TR, RF_Module:ST-SiP-LGA-86-11x7.3mm, symbol RF_Module:STM32WB5MMG
- removed U3: ~, Personal_Project:Button_KMR231GLFS, symbol Personal_Projects:Button_KMR231GLFS
- removed U5: USBLC6-2SC6, Package_TO_SOT_SMD:SOT-23-6, symbol Power_Protection:USBLC6-2SC6
- removed Z1: Diode_BZX84C6V2-7-F, Personal_Project:Diode_BZX84C6V2_SOT96P240X110-3N, symbol Personal_Projects:Diode_BZX84C6V2-7-F
Connections:
- no-connect marks 43 -> 0
Other:
- added sheet Interfaces (Interfaces.kicad_sch)
- added sheet Power_Management (Power_Management.kicad_sch)
- added sheet STM32WB5MMGH6TR (STM32WB5MMGH6TR.kicad_sch)
- added sheet USB (USB.kicad_sch)
- note removed: "BOOT0 Switch HIGH enables UART or I2C too allow programminng of the MCU LOW is start from flash memory"
- note removed: "Chip Select pin on general pin header"
- note removed: "EP is optional adhesive zone"
- note removed: "If shutdown capability is not required, connect EN to IN."
- note removed: "Input voltage range: 1.45V to 5.5V"
- note removed: "ON/OFF Switch"
- note removed: "Overvoltage protection for the PMOSFET VGS (VGS max is 8V)"
- note removed: "PH3_BOOT0 is tied low through an internal pull-down to enable start from flash memory. However, it can be tied high with a low resistive pull-up if required."
- note removed: "Polarity Protection"
- moved on the sheet: C2, U2
